File: pcb/matrix.kicad_pcb (KiCad board)
At the start: 2 copper layers, 57.4 x 47.1 mm, 69 parts, among them J1 Conn_01x02, J2 USB_C_Receptacle_USB2.0_14P, SW1 SW_Push, SW2 SW_Push, SW3 SW_Push, SW4 SW_Push, U1 ESP32-S3-MINI-1U, U2 AP2112K-3.3

Commit message: Update parts
Parts:
- U2: value AP2112K-3.3 -> XC6206PxxxMR; footprint Package_TO_SOT_SMD:SOT-23-5 -> Package_TO_SOT_SMD:SOT-23-3
- turned U2 to 0 degrees
Connections:
- U2 pad 1: Net-(J1-Pin_1) -> GND
- U2 pad 2: GND -> Net-(U1-3V3)
Routing:
- net Net-(J1-Pin_1): track 29.5 -> 26.1 mm
- net Net-(U1-3V3): track 69.1 -> 68.7 mm, vias 5 -> 6
